File: INJ.kicad_sch (KiCad schematic)
At the start: 6 parts, among them U501 VNLD5160TR-E, U502 VNLD5160TR-E

Commit message: test commit
Parts:
- renumbered U501 to U5001, U502 to U5002
Changed lines of the file:
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@@
 		(shape output)
 		(at 113.03 91.44 180)
-		(fields_autoplaced yes)
 		(effects
 			(font
@@
 		(shape output)
 		(at 113.03 64.77 180)
-		(fields_autoplaced yes)
 		(effects
 			(font
@@
 		(shape input)
 		(at 176.53 96.52 0)
-		(fields_autoplaced yes)
 		(effects
 			(font
@@
 		(shape input)
 		(at 176.53 69.85 0)
-		(fields_autoplaced yes)
 		(effects
 			(font
@@
 		(shape input)
 		(at 201.93 64.77 0)
-		(fields_autoplaced yes)
 		(effects
 			(font
@@
 		(shape input)
 		(at 201.93 91.44 0)
-		(fields_autoplaced yes)
 		(effects
 			(font
@@
 		(shape output)
 		(at 113.03 69.85 180)
-		(fields_autoplaced yes)
 		(effects
 			(font
@@
 		(shape output)
 		(at 113.03 96.52 180)
-		(fields_autoplaced yes)
 		(effects
 			(font
@@
 		(on_board yes)
 		(dnp no)
-		(property "Reference" "#PWR0503"
+		(property "Reference" "#PWR05003"
 			(at 166.37 86.36 0)
 			(effects
@@
 			(project "uaefi"
 				(path "/92ba706f-34f7-46cd-af88-2e1ff7aca489/908e7c38-dd3a-46e3-88c1-4637776bd8a8/cc5831c7-f9e2-4f1c-a3eb-62e5fbf6025f"
-					(reference "#PWR0503")
+					(reference "#PWR05003")
 					(unit 1)
 				)
@@
 		(on_board yes)
 		(dnp no)
-		(property "Reference" "#PWR0504"
+		(property "Reference" "#PWR05002"
 			(at 118.11 107.95 0)
 			(effects
@@
 			(project "uaefi"
 				(path "/92ba706f-34f7-46cd-af88-2e1ff7aca489/908e7c38-dd3a-46e3-88c1-4637776bd8a8/cc5831c7-f9e2-4f1c-a3eb-62e5fbf6025f"
-					(reference "#PWR0504")
+					(reference "#PWR05002")
 					(unit 1)
 				)
@@
 		(on_board yes)
 		(dnp no)
-		(property "Reference" "U501"
+		(property "Reference" "U5001"
 			(at 134.62 57.15 0)
 			(effects
@@
 			(project "uaefi"
 				(path "/92ba706f-34f7-46cd-af88-2e1ff7aca489/908e7c38-dd3a-46e3-88c1-4637776bd8a8/cc5831c7-f9e2-4f1c-a3eb-62e5fbf6025f"
-					(reference "U501")
+					(reference "U5001")
 					(unit 1)
 				)
@@
 			(project "alphax_8ch"
 				(path "/92ba706f-34f7-46cd-af88-2e1ff7aca489/908e7c38-dd3a-46e3-88c1-4637776bd8a8/cc5831c7-f9e2-4f1c-a3eb-62e5fbf6025f"
-					(reference "R503")
+					(reference "R5004")
 					(unit 1)
 				)
@@
 		(on_board yes)
 		(dnp no)
-		(property "Reference" "U502"
+		(property "Reference" "U5002"
 			(at 134.62 83.82 0)
 			(effects
@@
 			(project "uaefi"
 				(path "/92ba706f-34f7-46cd-af88-2e1ff7aca489/908e7c38-dd3a-46e3-88c1-4637776bd8a8/cc5831c7-f9e2-4f1c-a3eb-62e5fbf6025f"
-					(reference "U502")
+					(reference "U5002")
 					(unit 1)
 				)
@@
 		(on_board yes)
 		(dnp no)
-		(property "Reference" "#PWR0506"
+		(property "Reference" "#PWR05004"
 			(at 166.37 113.03 0)
 			(effects
@@
 			(project "uaefi"
 				(path "/92ba706f-34f7-46cd-af88-2e1ff7aca489/908e7c38-dd3a-46e3-88c1-4637776bd8a8/cc5831c7-f9e2-4f1c-a3eb-62e5fbf6025f"
-					(reference "#PWR0506")
+					(reference "#PWR05004")
 					(unit 1)
 				)
@@
 		(on_board yes)
 		(dnp no)
-		(property "Reference" "#PWR0502"
+		(property "Reference" "#PWR05005"
 			(at 189.23 81.28 0)
 			(effects
@@
 			(project "uaefi"
 				(path "/92ba706f-34f7-46cd-af88-2e1ff7aca489/908e7c38-dd3a-46e3-88c1-4637776bd8a8/cc5831c7-f9e2-4f1c-a3eb-62e5fbf6025f"
-					(reference "#PWR0502")
+					(reference "#PWR05005")
 					(unit 1)
 				)
@@
 		(on_board yes)
 		(dnp no)
-		(property "Reference" "#PWR0505"
+		(property "Reference" "#PWR05006"
 			(at 189.23 107.95 0)
 			(effects
@@
 			(project "uaefi"
 				(path "/92ba706f-34f7-46cd-af88-2e1ff7aca489/908e7c38-dd3a-46e3-88c1-4637776bd8a8/cc5831c7-f9e2-4f1c-a3eb-62e5fbf6025f"
-					(reference "#PWR0505")
+					(reference "#PWR05006")
 					(unit 1)
 				)
@@
 			(project "alphax_8ch"
 				(path "/92ba706f-34f7-46cd-af88-2e1ff7aca489/908e7c38-dd3a-46e3-88c1-4637776bd8a8/cc5831c7-f9e2-4f1c-a3eb-62e5fbf6025f"
-					(reference "R502")
+					(reference "R5001")
 					(unit 1)
 				)
@@
 			(project "alphax_8ch"
 				(path "/92ba706f-34f7-46cd-af88-2e1ff7aca489/908e7c38-dd3a-46e3-88c1-4637776bd8a8/cc5831c7-f9e2-4f1c-a3eb-62e5fbf6025f"
-					(reference "R504")
+					(reference "R5002")
 					(unit 1)
 				)
@@
 			(project "alphax_8ch"
 				(path "/92ba706f-34f7-46cd-af88-2e1ff7aca489/908e7c38-dd3a-46e3-88c1-4637776bd8a8/cc5831c7-f9e2-4f1c-a3eb-62e5fbf6025f"
-					(reference "R501")
+					(reference "R5003")
 					(unit 1)
 				)
@@
 		(on_board yes)
 		(dnp no)
-		(property "Reference" "#PWR0501"
+		(property "Reference" "#PWR05001"
 			(at 118.11 81.28 0)
 			(effects
@@
 			(project "uaefi"
 				(path "/92ba706f-34f7-46cd-af88-2e1ff7aca489/908e7c38-dd3a-46e3-88c1-4637776bd8a8/cc5831c7-f9e2-4f1c-a3eb-62e5fbf6025f"
-					(reference "#PWR0501")
-					(unit 1)
-				)
+					(reference "#PWR05001")
+					(unit 1)
+				)
