File: conn.kicad_sch (KiCad schematic)
At the start: 3 parts, among them J201 Conn_02x03_Top_Bottom, J203 Conn_02x12_Top_Bottom, P201 134pin_7-967288-1_KC5

Commit message: test commit
Parts:
- renumbered J203 to J2001, J201 to J2002, P201 to P2001

Commit message: Initial schematic
Parts:
- added F2001, F2002, F2003, F2004: 10A, hellen-one-common:36911600000, symbol hellen-one-common:Fuse-Pad-Pad
- added JP2001, JP2003, JP2004, JP2005, JP2010, JP2011, JP2012: Jumper_2_Bridged, Jumper:SolderJumper-2_P1.3mm_Bridged_RoundedPad1.0x1.5mm, symbol Jumper:Jumper_2_Bridged
- added JP2002, JP2006, JP2007, JP2008, JP2009: Jumper_2_Open, hellen-one-common:PAD-0805-PAD, symbol hellen-one-common:Jumper-Pad-Pad
- J2001: symbol Connector_Generic:Conn_02x12_Top_Bottom -> Connector_Generic:Conn_01x24
- P2001: now left out of the parts list
Connections:
- net ECU_NBO2pre_H+ is gone; now on net +12V_RAW: P2001.224 (Pin_224)
- net +12V_RAW: now also J2001.6 (Pin_6), J2002.1 (Pin_1), P2001.303 (Pin_303), P2001.304 (Pin_304), P2001.305 (Pin_305), P2001.306 (Pin_306), P2001.316 (Pin_316), P2001.343 (Pin_343), P2001.352 (Pin_352)
- net ECU_CANH: now also JP2011.2 (B)
- net ECU_CANL: now also JP2012.2 (B)
- net ECU_MAINREL: now also JP2002.2
- net ECU_NBO2pre_H-: now also JP2003.2 (B)
- net ECU_NBO2pre_SIG+: now also JP2001.2 (B)
- net ECU_NBO2pre_SIG-: now also JP2004.2 (B)
- net GND: now also J2001.12 (Pin_12), J2001.16 (Pin_16), J2001.17 (Pin_17), J2001.21 (Pin_21), J2001.7 (Pin_7), JP2004.1 (A); no longer P2001.307 (Pin_307), P2001.309 (Pin_309)
- net IGN_OUT1: now also F2002.1; no longer P2001.506 (Pin_506)
- net IGN_OUT2: now also F2001.1; no longer P2001.504 (Pin_504)
- net IGN_OUT3: now also F2003.1; no longer P2001.508 (Pin_508)
- net IGN_OUT4: now also F2004.1; no longer P2001.509 (Pin_509)
- net INJ_OUT1: now also JP2009.1; no longer P2001.351 (Pin_351)
- net INJ_OUT2: now also JP2008.1; no longer P2001.350 (Pin_350)
- net INJ_OUT3: now also JP2007.1; no longer P2001.349 (Pin_349)
- net INJ_OUT4: now also JP2006.1; no longer P2001.348 (Pin_348)
- net KNOCK1: now also P2001.332 (Pin_332); no longer P2001.331 (Pin_331)
- net KNOCK2: now also P2001.331 (Pin_331); no longer P2001.332 (Pin_332)
- net LIN: now also JP2010.1 (A); no longer P2001.206 (Pin_206), P2001.432 (Pin_432)
- net CRANK_FB: now reaches P2001.312 (Pin_312)
- net CRANK_FB: now also P2001.402 (Pin_402)
- net CHARGE: now reaches P2001.313 (Pin_313)
- net CHARGE: now also P2001.401 (Pin_401)
- net OIL_P: now reaches P2001.326 (Pin_326)
- net OIL_P: now also P2001.411 (Pin_411), JP2005.2 (B)
- net +5VA: now reaches P2001.327 (Pin_327)
- net +5VA: now also J2001.19 (Pin_19), J2001.20 (Pin_20), P2001.346 (Pin_346)
- net AIN.CLT: now reaches P2001.328 (Pin_328)
- net AIN.IAT: now reaches P2001.329 (Pin_329)
- net AIN.MAF: now reaches P2001.330 (Pin_330)
- net AIN.TPS: now reaches P2001.333 (Pin_333)
- net DIN.CPS: now reaches P2001.335 (Pin_335)
- net DIN.CMP: now reaches P2001.338 (Pin_338)
- net F_OLN: now reaches P2001.339 (Pin_339)
- net F_OLN: now also P2001.421 (Pin_421)
- net PP.IACVO: now reaches P2001.340 (Pin_340)
- net PP.IACVC: now reaches P2001.341 (Pin_341)
- net OUTLS.FTVV: now reaches P2001.344 (Pin_344)
- net OUTLS.DISA: now reaches P2001.345 (Pin_345)
- net USB.DP: now reaches J2001.1 (Pin_1)
- net USB.VBUS: now reaches J2001.11 (Pin_11)
- net CAN2L: now reaches J2001.13 (Pin_13)
- net CAN2H: now reaches J2001.14 (Pin_14)
- net KNOCK_HP2: now reaches J2001.15 (Pin_15)
- net AIN.MAP: now reaches J2001.18 (Pin_18)
- net USB.DM: now reaches J2001.2 (Pin_2)
- net EXTIN1: now reaches J2001.22 (Pin_22)
- net EXTIN2: now reaches J2001.23 (Pin_23)
- net CAN1L: now reaches J2001.3 (Pin_3)
- net CAN1L: now also JP2012.1 (A)
- net CAN1H: now reaches J2001.4 (Pin_4)
- net CAN1H: now also JP2011.1 (A)
- net KNOCK_HP1: now reaches J2001.5 (Pin_5)
- net OUTLS.SLP: now reaches P2001.403 (Pin_403)
- net PP.FAN: now reaches P2001.404 (Pin_404)
- net OUTLS.EKP: now reaches P2001.410 (Pin_410)
- net PP.FTD: now reaches P2001.417 (Pin_417)
- net DIN.RRWS: now reaches P2001.422 (Pin_422)
- net OUTLS.KOREL: now reaches P2001.429 (Pin_429)
- net DIN.EWS: now reaches P2001.433 (Pin_433)
- net AIN.TRAD: now reaches P2001.439 (Pin_439)
- new net: JP2006.2, P2001.348 (Pin_348)
- new net: F2001.2, P2001.504 (Pin_504)
- new net: F2003.2, P2001.508 (Pin_508)
- new net: F2002.2, P2001.506 (Pin_506)
- new net: F2004.2, P2001.509 (Pin_509)
- new net: JP2007.2, P2001.349 (Pin_349)
- new net: JP2008.2, P2001.350 (Pin_350)
- new net: JP2009.2, P2001.351 (Pin_351)
- new net AIN.NBO2: JP2001.1 (A)
- new net DIN.OPS: JP2005.1 (A)
- new net ECU_LIN: JP2010.2 (B), P2001.206 (Pin_206), P2001.432 (Pin_432)
- new net NBO2H: JP2003.1 (A)
- new net OUTLS.MREL: JP2002.1
- new net OUTLS.SLV: P2001.307 (Pin_307)
- new net OUTLS.THERMO: P2001.309 (Pin_309)
- no-connect marks 26 -> 59
Other:
- note added: "Narrowband O2 not connected, use wideband on external plug"
- moved on the sheet: J2001, J2002, P2001A, P2001B, P2001C, P2001D, P2001E

Commit message: Initial schematic
Parts:
- P2001: now in the parts list
Changed lines of the file:
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@@
 		(unit 5)
 		(exclude_from_sim no)
-		(in_bom no)
+		(in_bom yes)
 		(on_board yes)
 		(dnp no)
@@
 		(unit 3)
 		(exclude_from_sim no)
-		(in_bom no)
+		(in_bom yes)
 		(on_board yes)
 		(dnp no)
@@
 		(unit 2)
 		(exclude_from_sim no)
-		(in_bom no)
+		(in_bom yes)
 		(on_board yes)
 		(dnp no)
@@
 		(unit 4)
 		(exclude_from_sim no)
-		(in_bom no)
+		(in_bom yes)
 		(on_board yes)
 		(dnp no)
@@
 		(unit 1)
 		(exclude_from_sim no)
-		(in_bom no)
+		(in_bom yes)
 		(on_board yes)
 		(dnp no)
