File: outls.kicad_sch (KiCad schematic)
At the start: 6 parts, among them U5001 VNLD5160TR-E, U5002 VNLD5160TR-E

Commit message: Initial schematic
Parts:
- removed R5001, R5002, R5003, R5004: 4.7k, hellen-one-common:R0603, symbol hellen-one-common:Res
- removed U5001, U5002: VNLD5160TR-E, Package_SO:SOIC-8_3.9x4.9mm_P1.27mm, symbol chips:VNLD5160
- added R7001, R7002, R7003, R7004: 4.7k, hellen-one-common:R0603, symbol hellen-one-common:Res
- added U7001, U7002: VNLD5160TR-E, Package_SO:SOIC-8_3.9x4.9mm_P1.27mm, symbol chips:VNLD5160
Connections:
- net GND: now also R7001.1, R7002.1, R7003.1, R7004.1, U7001.5 (S2), U7001.7 (S1), U7002.5 (S2), U7002.7 (S1)
- net IN1: now also R7003.2, U7001.1 (IN1)
- net IN2: now also R7001.2, U7001.3 (IN2)
- net IN3: now also R7004.2, U7002.1 (IN1)
- net IN4: now also R7002.2, U7002.3 (IN2)
- net OUT1: now also U7001.8 (D1)
- net OUT2: now also U7001.6 (D2)
- net OUT3: now also U7002.8 (D1)
- net OUT4: now also U7002.6 (D2)
Other:
- company: rusEFI.com -> (none)
- title: UAEFI -> (none)

Commit message: Initial schematic
Parts:
- renumbered R7001 to R8001, R7002 to R8002, R7003 to R8003, R7004 to R8004, U7001 to U8001, U7002 to U8002
Changed lines of the file:
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@@
 		(on_board yes)
 		(dnp no)
-		(property "Reference" "R7004"
+		(property "Reference" "R8004"
 			(at 163.83 99.06 0)
 			(effects
@@
 		(on_board yes)
 		(dnp no)
-		(property "Reference" "#PWR07004"
+		(property "Reference" "#PWR08004"
 			(at 143.51 115.57 0)
 			(effects
@@
 		(on_board yes)
 		(dnp no)
-		(property "Reference" "#PWR07005"
+		(property "Reference" "#PWR08005"
 			(at 166.37 83.82 0)
 			(effects
@@
 		(on_board yes)
 		(dnp no)
-		(property "Reference" "R7003"
+		(property "Reference" "R8003"
 			(at 163.83 72.39 0)
 			(effects
@@
 		(on_board yes)
 		(dnp no)
-		(property "Reference" "U7001"
+		(property "Reference" "U8001"
 			(at 111.76 59.69 0)
 			(effects
@@
 		(on_board yes)
 		(dnp no)
-		(property "Reference" "#PWR07006"
+		(property "Reference" "#PWR08006"
 			(at 166.37 110.49 0)
 			(effects
@@
 		(on_board yes)
 		(dnp no)
-		(property "Reference" "R7001"
+		(property "Reference" "R8001"
 			(at 140.97 77.47 0)
 			(effects
@@
 		(on_board yes)
 		(dnp no)
-		(property "Reference" "#PWR07001"
+		(property "Reference" "#PWR08001"
 			(at 95.25 83.82 0)
 			(effects
@@
 		(on_board yes)
 		(dnp no)
-		(property "Reference" "R7002"
+		(property "Reference" "R8002"
 			(at 140.97 104.14 0)
 			(effects
@@
 		(on_board yes)
 		(dnp no)
-		(property "Reference" "#PWR07003"
+		(property "Reference" "#PWR08003"
 			(at 143.51 88.9 0)
 			(effects
@@
 		(on_board yes)
 		(dnp no)
-		(property "Reference" "U7002"
+		(property "Reference" "U8002"
 			(at 111.76 86.36 0)
 			(effects
@@
 		(on_board yes)
 		(dnp no)
-		(property "Reference" "#PWR07002"
+		(property "Reference" "#PWR08002"
 			(at 95.25 110.49 0)
 			(effects
