File: rusefi.kicad_sch (KiCad schematic)
At the start: 9 parts, among them J301 USB_B, M301 Module:mega-mcu100/0.3, M302 Module-can-0.1, M303 Module-wbo-0.5, M304 Module-lin-0.1, M306 Module-power_12and5V-0.2

Commit message: test commit
Parts:
- renumbered BT301 to BT3001, D301 to D3001, J301 to J3001, JP301 to JP3001, M306 to M3001, M301 to M3002, M302 to M3003, M303 to M3004, M304 to M3005

Commit message: Initial schematic
Parts:
- added TP3001, TP3002, TP3003, TP3004, TP3005, TP3006, TP3007, TP3008, TP3009, TP3010: TestPoint, TestPoint:TestPoint_Keystone_5000-5004_Miniature, symbol Connector:TestPoint
- renumbered M3004 to M3003, M3003 to M3004
Connections:
- net +12V_RAW: now also M3005.N1 (12V), M3005.V1 (12V)
- net +3.3VA: now also M3004.V2 (CAN_VIO)
- net +5VA: now also M3003.W1 (V5_IN), M3004.V1 (V5), M3005.V3 (5V)
- net GND: now also M3001.S1 (GND), M3003.E6 (LSU_H-), M3003.G (GND), M3004.E1 (GND), M3005.E1 (GND), M3005.S1 (GND)
- net CAN2L: now reaches M3004.S1 (CANL)
- net CAN2H: now reaches M3004.S2 (CANH)
- net OUT LS1/IN4: now reaches M3002.E10 (OUT_INJ8_(PD12))
- net OUT LS1/IN3: now reaches M3002.E11 (OUT_INJ7_(PD15))
- net OUT LS1/IN2: now reaches M3002.E12 (OUT_INJ6_(PA8))
- net OUT LS1/IN1: now reaches M3002.E13 (OUT_INJ5_(PD2))
- net OUT PP/IN1: now reaches M3002.E18 (OUT_PWM1_(PD13))
- net OUT PP/IN2: now reaches M3002.E19 (OUT_PWM2_(PC6))
- net OUT PP1/IN1: now reaches M3002.E20 (OUT_PWM3_(PC7))
- net OUT PP1/IN2: now reaches M3002.E21 (OUT_PWM4_(PC8))
- net NBO2H/IN: now reaches M3002.E22 (OUT_PWM5_(PC9))
- net at M3002.E23 (OUT_PWM6_(PD14)): now also TP3007.1
- net at M3002.N16 (BOOT0): now also TP3010.1
- net at M3002.N4 (USBID_(PA10)): now also TP3008.1
- net at M3002.N7 (nReset): now also TP3009.1
- net EXTIN2: now reaches M3002.S1 (IN_D4_(PE15))
- net AIN.NBO2: now reaches M3002.S10 (IN_O2S2_(PA1))
- net at M3002.S11 (IN_O2S_/_CAN_WAKEUP_(PA0)): now also TP3002.1
- net at M3002.S12 (IN_MAP2_(PC1)): now also TP3003.1
- net DIN.CPS: now reaches M3002.S14 (IN_CRANK_(PB1))
- net DIN.CMP: now reaches M3002.S16 (IN_CAM_(PA6))
- net DIN.RRWS: now reaches M3002.S17 (IN_VSS_(PE11))
- net at M3002.S19 (IN_PPS_(PA3)): now also TP3006.1
- net EXTIN1: now reaches M3002.S2 (IN_D3_(PE14))
- net DIN.EWS: now reaches M3002.S3 (IN_D2_(PE13))
- net DIN.OPS: now reaches M3002.S4 (IN_D1_(PE12))
- net at M3002.S5 (VREF2): now also TP3005.1
- net at M3002.S6 (IN_AUX4_(PC5)): now also TP3004.1
- net at M3002.W13 (V33_REF): now also TP3001.1
- net OUT LS/IN4: now reaches M3002.W3 (IGN8_(PE6))
- net OUT LS/IN3: now reaches M3002.W4 (IGN7_(PB9))
- net OUT LS/IN2: now reaches M3002.W5 (IGN6_(PB8))
- net OUT LS/IN1: now reaches M3002.W6 (IGN5_(PE2))
- net AIN.OILTEMP1 renamed AIN.MAF
- net AIN.OILTEMP2 renamed AIN.TRAD
- net CANH renamed CAN1H
- net CANL renamed CAN1L
- net Ignition/IN1 renamed IGN1
- net Ignition/IN2 renamed IGN2
- net Ignition/IN3 renamed IGN3
- net Ignition/IN4 renamed IGN4
- net Injection/IN1 renamed INJ1
- net Injection/IN2 renamed INJ2
- net Injection/IN3 renamed INJ3
- net Injection/IN4 renamed INJ4
- no-connect marks 13 -> 25
Other:
- added sheet NBO2H (nbo2h.kicad_sch)
- added sheet OUT LS (outls.kicad_sch)
- added sheet OUT LS1 (outls.kicad_sch)
- added sheet OUT PP (outpp.kicad_sch)
- added sheet OUT PP1 (outpp.kicad_sch)
- sheet KnockAmps ports: added KNOCK_HP[1..2]; removed KNOCK_HP1, KNOCK_HP2
- note added: "Replace resistors for AUX3 with same setup as KNOCK"
- moved on the sheet: M3004

Commit message: inital schamatic
Parts:
- TP3001, TP3002, TP3003, TP3004, TP3005, TP3006, TP3007, TP3008, TP3009, TP3010: now in the parts list
Changed lines of the file:
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@@
 		(unit 1)
 		(exclude_from_sim no)
-		(in_bom no)
+		(in_bom yes)
 		(on_board yes)
 		(dnp no)
@@
 		(unit 1)
 		(exclude_from_sim no)
-		(in_bom no)
+		(in_bom yes)
 		(on_board yes)
 		(dnp no)
@@
 		(unit 1)
 		(exclude_from_sim no)
-		(in_bom no)
+		(in_bom yes)
 		(on_board yes)
 		(dnp no)
@@
 		(unit 1)
 		(exclude_from_sim no)
-		(in_bom no)
+		(in_bom yes)
 		(on_board yes)
 		(dnp no)
@@
 		(unit 1)
 		(exclude_from_sim no)
-		(in_bom no)
+		(in_bom yes)
 		(on_board yes)
 		(dnp no)
@@
 		(unit 1)
 		(exclude_from_sim no)
-		(in_bom no)
+		(in_bom yes)
 		(on_board yes)
 		(dnp no)
@@
 		(unit 1)
 		(exclude_from_sim no)
-		(in_bom no)
+		(in_bom yes)
 		(on_board yes)
 		(dnp no)
@@
 		(unit 1)
 		(exclude_from_sim no)
-		(in_bom no)
+		(in_bom yes)
 		(on_board yes)
 		(dnp no)
@@
 		(unit 1)
 		(exclude_from_sim no)
-		(in_bom no)
+		(in_bom yes)
 		(on_board yes)
 		(dnp no)
@@
 		(unit 1)
 		(exclude_from_sim no)
-		(in_bom no)
-		(on_board yes)
-		(dnp no)
+		(in_bom yes)
+		(on_board yes)
+		(dnp no)
