File: IGN.kicad_sch (KiCad schematic)
At the start: 16 parts

Commit message: test commit
Parts:
- renumbered F401 to F4001, F403 to F4002, F404 to F4003, F402 to F4004
Changed lines of the file:
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@@
 		(shape output)
 		(at 113.03 64.77 180)
-		(fields_autoplaced yes)
 		(effects
 			(font
@@
 		(shape output)
 		(at 113.03 120.65 180)
-		(fields_autoplaced yes)
 		(effects
 			(font
@@
 		(shape input)
 		(at 143.51 97.79 0)
-		(fields_autoplaced yes)
 		(effects
 			(font
@@
 		(shape output)
 		(at 113.03 92.71 180)
-		(fields_autoplaced yes)
 		(effects
 			(font
@@
 		(shape input)
 		(at 143.51 125.73 0)
-		(fields_autoplaced yes)
 		(effects
 			(font
@@
 		(shape input)
 		(at 143.51 69.85 0)
-		(fields_autoplaced yes)
 		(effects
 			(font
@@
 		(shape output)
 		(at 160.02 64.77 180)
-		(fields_autoplaced yes)
 		(effects
 			(font
@@
 		(shape input)
 		(at 190.5 69.85 0)
-		(fields_autoplaced yes)
 		(effects
 			(font
@@
 			(project "hellen-hyundai-pb-154"
 				(path "/92ba706f-34f7-46cd-af88-2e1ff7aca489/908e7c38-dd3a-46e3-88c1-4637776bd8a8/9b0b4a5a-9407-413d-9bb4-c60fbda7f3a8"
-					(reference "Q404")
+					(reference "Q4003")
 					(unit 1)
 				)
@@
 			(project "proteus81harley"
 				(path "/92ba706f-34f7-46cd-af88-2e1ff7aca489/908e7c38-dd3a-46e3-88c1-4637776bd8a8/9b0b4a5a-9407-413d-9bb4-c60fbda7f3a8"
-					(reference "R403")
+					(reference "R4001")
 					(unit 1)
 				)
@@
 			(project "proteus81harley"
 				(path "/92ba706f-34f7-46cd-af88-2e1ff7aca489/908e7c38-dd3a-46e3-88c1-4637776bd8a8/9b0b4a5a-9407-413d-9bb4-c60fbda7f3a8"
-					(reference "R402")
+					(reference "R4008")
 					(unit 1)
 				)
@@
 			(project "proteus81harley"
 				(path "/92ba706f-34f7-46cd-af88-2e1ff7aca489/908e7c38-dd3a-46e3-88c1-4637776bd8a8/9b0b4a5a-9407-413d-9bb4-c60fbda7f3a8"
-					(reference "R406")
+					(reference "R4002")
 					(unit 1)
 				)
@@
 			(project "hellen-hyundai-pb-154"
 				(path "/92ba706f-34f7-46cd-af88-2e1ff7aca489/908e7c38-dd3a-46e3-88c1-4637776bd8a8/9b0b4a5a-9407-413d-9bb4-c60fbda7f3a8"
-					(reference "#PWR0404")
+					(reference "#PWR04003")
 					(unit 1)
 				)
@@
 			(project "proteus81harley"
 				(path "/92ba706f-34f7-46cd-af88-2e1ff7aca489/908e7c38-dd3a-46e3-88c1-4637776bd8a8/9b0b4a5a-9407-413d-9bb4-c60fbda7f3a8"
-					(reference "R401")
+					(reference "R4004")
 					(unit 1)
 				)
@@
 			(project "hellen-hyundai-pb-154"
 				(path "/92ba706f-34f7-46cd-af88-2e1ff7aca489/908e7c38-dd3a-46e3-88c1-4637776bd8a8/9b0b4a5a-9407-413d-9bb4-c60fbda7f3a8"
-					(reference "Q401")
+					(reference "Q4001")
 					(unit 1)
 				)
@@
 			(project "proteus81harley"
 				(path "/92ba706f-34f7-46cd-af88-2e1ff7aca489/908e7c38-dd3a-46e3-88c1-4637776bd8a8/9b0b4a5a-9407-413d-9bb4-c60fbda7f3a8"
-					(reference "R408")
+					(reference "R4003")
 					(unit 1)
 				)
@@
 			(project "hellen-hyundai-pb-154"
 				(path "/92ba706f-34f7-46cd-af88-2e1ff7aca489/908e7c38-dd3a-46e3-88c1-4637776bd8a8/9b0b4a5a-9407-413d-9bb4-c60fbda7f3a8"
-					(reference "Q403")
+					(reference "Q4002")
 					(unit 1)
 				)
@@
 			(project "hellen-hyundai-pb-154"
 				(path "/92ba706f-34f7-46cd-af88-2e1ff7aca489/908e7c38-dd3a-46e3-88c1-4637776bd8a8/9b0b4a5a-9407-413d-9bb4-c60fbda7f3a8"
-					(reference "#PWR0401")
+					(reference "#PWR04001")
 					(unit 1)
 				)
@@
 		(on_board yes)
 		(dnp no)
-		(property "Reference" "F401"
+		(property "Reference" "F4001"
 			(at 139.7 67.31 90)
 			(effects
@@
 			(project "uaefi"
 				(path "/92ba706f-34f7-46cd-af88-2e1ff7aca489/908e7c38-dd3a-46e3-88c1-4637776bd8a8/9b0b4a5a-9407-413d-9bb4-c60fbda7f3a8"
-					(reference "F401")
+					(reference "F4001")
 					(unit 1)
 				)
@@
 			(project "hellen-hyundai-pb-154"
 				(path "/92ba706f-34f7-46cd-af88-2e1ff7aca489/908e7c38-dd3a-46e3-88c1-4637776bd8a8/9b0b4a5a-9407-413d-9bb4-c60fbda7f3a8"
-					(reference "Q402")
+					(reference "Q4004")
 					(unit 1)
 				)
@@
 		(on_board yes)
 		(dnp no)
-		(property "Reference" "F403"
+		(property "Reference" "F4002"
 			(at 139.7 95.25 90)
 			(effects
@@
 			(project "uaefi"
 				(path "/92ba706f-34f7-46cd-af88-2e1ff7aca489/908e7c38-dd3a-46e3-88c1-4637776bd8a8/9b0b4a5a-9407-413d-9bb4-c60fbda7f3a8"
-					(reference "F403")
+					(reference "F4002")
 					(unit 1)
 				)
@@
 			(project "hellen-hyundai-pb-154"
 				(path "/92ba706f-34f7-46cd-af88-2e1ff7aca489/908e7c38-dd3a-46e3-88c1-4637776bd8a8/9b0b4a5a-9407-413d-9bb4-c60fbda7f3a8"
-					(reference "#PWR0402")
+					(reference "#PWR04004")
 					(unit 1)
 				)
@@
 			(project "proteus81harley"
 				(path "/92ba706f-34f7-46cd-af88-2e1ff7aca489/908e7c38-dd3a-46e3-88c1-4637776bd8a8/9b0b4a5a-9407-413d-9bb4-c60fbda7f3a8"
-					(reference "R405")
+					(reference "R4005")
 					(unit 1)
 				)
@@
 			(project "proteus81harley"
 				(path "/92ba706f-34f7-46cd-af88-2e1ff7aca489/908e7c38-dd3a-46e3-88c1-4637776bd8a8/9b0b4a5a-9407-413d-9bb4-c60fbda7f3a8"
-					(reference "R404")
+					(reference "R4007")
 					(unit 1)
 				)
@@
 			(project "hellen-hyundai-pb-154"
 				(path "/92ba706f-34f7-46cd-af88-2e1ff7aca489/908e7c38-dd3a-46e3-88c1-4637776bd8a8/9b0b4a5a-9407-413d-9bb4-c60fbda7f3a8"
-					(reference "#PWR0403")
+					(reference "#PWR04002")
 					(unit 1)
 				)
@@
 			(project "proteus81harley"
 				(path "/92ba706f-34f7-46cd-af88-2e1ff7aca489/908e7c38-dd3a-46e3-88c1-4637776bd8a8/9b0b4a5a-9407-413d-9bb4-c60fbda7f3a8"
-					(reference "R407")
+					(reference "R4006")
 					(unit 1)
 				)
@@
 		(on_board yes)
 		(dnp no)
-		(property "Reference" "F402"
+		(property "Reference" "F4004"
 			(at 186.69 67.31 90)
 			(effects
@@
 			(project "uaefi"
 				(path "/92ba706f-34f7-46cd-af88-2e1ff7aca489/908e7c38-dd3a-46e3-88c1-4637776bd8a8/9b0b4a5a-9407-413d-9bb4-c60fbda7f3a8"
-					(reference "F402")
+					(reference "F4004")
 					(unit 1)
 				)
@@
 		(on_board yes)
 		(dnp no)
-		(property "Reference" "F404"
+		(property "Reference" "F4003"
 			(at 139.7 123.19 90)
 			(effects
@@
 			(project "uaefi"
 				(path "/92ba706f-34f7-46cd-af88-2e1ff7aca489/908e7c38-dd3a-46e3-88c1-4637776bd8a8/9b0b4a5a-9407-413d-9bb4-c60fbda7f3a8"
-					(reference "F404")
-					(unit 1)
-				)
+					(reference "F4003")
+					(unit 1)
+				)

Commit message: Initial schematic
Parts:
- removed R14 (x4): 0, Resistor_SMD:R_2512_6332Metric, symbol hellen-one-common:Res
- added JP4001, JP4002, JP4003, JP4004: Jumper_2_Open, hellen-one-common:PAD-0805-PAD, symbol hellen-one-common:Jumper-Pad-Pad
- Q? (x4): MyComment DNP -> (none)
Connections:
- net OUT1: now also JP4001.1
- net OUT2: now also JP4002.1
- net OUT3: now also JP4003.1
- net OUT4: now also JP4004.1
- net at F4001.1, R7.2: now also JP4001.2
- net at F4004.1, R7.2: now also JP4004.2
- net at F4002.1, R7.2: now also JP4002.2
- net at F4003.1, R7.2: now also JP4003.2
Other:
- note added: "Dumb coils use Q4001-Q4004, R4001, R4002, R4003, R4007 COP or external igniter use R4004, R4005, R4006, R4008"
- note removed: "Remove R20-R22, R26-R28, and install Q7-Q12 for use with dumb coils"

Commit message: adjusted BOM
Parts:
- Q? (x4): LCSC (none) -> C462128
Changed lines of the file:
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@@
 			)
 		)
-		(property "LCSC" ""
+		(property "LCSC" "C462128"
 			(at 120.65 125.73 0)
 			(effects
@@
 			)
 		)
-		(property "LCSC" ""
+		(property "LCSC" "C462128"
 			(at 120.65 69.85 0)
 			(effects
@@
 			)
 		)
-		(property "LCSC" ""
+		(property "LCSC" "C462128"
 			(at 120.65 97.79 0)
 			(effects
@@
 			)
 		)
-		(property "LCSC" ""
+		(property "LCSC" "C462128"
 			(at 167.64 69.85 0)
 			(effects
