File: knockamps.kicad_sch (KiCad schematic)
At the start: 6 parts, among them M601 Module-knock-0.2, M602 Module-knock-0.2, U601 MCP6002-xSN

Commit message: test commit
Parts:
- renumbered C601 to C6001, C602 to C6002, C603 to C6003, M601 to M6001, M602 to M6002, U601 to U6001
Changed lines of the file:
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@@
 	(label "KNOCK2"
 		(at 60.96 127 0)
-		(fields_autoplaced yes)
 		(effects
 			(font
@@
 	(label "KNOCK1"
 		(at 60.96 45.72 0)
-		(fields_autoplaced yes)
 		(effects
 			(font
@@
 		(shape output)
 		(at 246.38 127 0)
-		(fields_autoplaced yes)
 		(effects
 			(font
@@
 		(shape output)
 		(at 246.38 73.66 0)
-		(fields_autoplaced yes)
 		(effects
 			(font
@@
 		(shape output)
 		(at 246.38 21.59 0)
-		(fields_autoplaced yes)
 		(effects
 			(font
@@
 		(shape input)
 		(at 40.64 137.16 180)
-		(fields_autoplaced yes)
 		(effects
 			(font
@@
 		(shape output)
 		(at 246.38 45.72 0)
-		(fields_autoplaced yes)
 		(effects
 			(font
@@
 		(shape output)
 		(at 246.38 99.06 0)
-		(fields_autoplaced yes)
 		(effects
 			(font
@@
 		(dnp no)
 		(fields_autoplaced yes)
-		(property "Reference" "#PWR0601"
+		(property "Reference" "#PWR06003"
 			(at 97.79 31.75 0)
 			(effects
@@
 			(project ""
 				(path "/92ba706f-34f7-46cd-af88-2e1ff7aca489/908e7c38-dd3a-46e3-88c1-4637776bd8a8/fd7b0d96-5428-4c2c-8651-d380ef93928b"
-					(reference "#PWR0601")
+					(reference "#PWR06003")
 					(unit 1)
 				)
@@
 		(dnp no)
 		(fields_autoplaced yes)
-		(property "Reference" "M601"
+		(property "Reference" "M6001"
 			(at 122.908 39.575 0)
 			(effects
@@
 			(project "hellenbms46"
 				(path "/92ba706f-34f7-46cd-af88-2e1ff7aca489/908e7c38-dd3a-46e3-88c1-4637776bd8a8/fd7b0d96-5428-4c2c-8651-d380ef93928b"
-					(reference "M601")
+					(reference "M6001")
 					(unit 1)
 				)
@@
 		(dnp no)
 		(fields_autoplaced yes)
-		(property "Reference" "U601"
+		(property "Reference" "U6001"
 			(at 164.465 85.1478 0)
 			(effects
@@
 			(project ""
 				(path "/92ba706f-34f7-46cd-af88-2e1ff7aca489/908e7c38-dd3a-46e3-88c1-4637776bd8a8/fd7b0d96-5428-4c2c-8651-d380ef93928b"
-					(reference "U601")
+					(reference "U6001")
 					(unit 3)
 				)
@@
 		(dnp no)
 		(fields_autoplaced yes)
-		(property "Reference" "#PWR0602"
+		(property "Reference" "#PWR06004"
 			(at 97.79 113.03 0)
 			(effects
@@
 			(project ""
 				(path "/92ba706f-34f7-46cd-af88-2e1ff7aca489/908e7c38-dd3a-46e3-88c1-4637776bd8a8/fd7b0d96-5428-4c2c-8651-d380ef93928b"
-					(reference "#PWR0602")
+					(reference "#PWR06004")
 					(unit 1)
 				)
@@
 		(dnp no)
 		(fields_autoplaced yes)
-		(property "Reference" "C601"
+		(property "Reference" "C6001"
 			(at 156.591 85.1478 0)
 			(effects
@@
 			(project ""
 				(path "/92ba706f-34f7-46cd-af88-2e1ff7aca489/908e7c38-dd3a-46e3-88c1-4637776bd8a8/fd7b0d96-5428-4c2c-8651-d380ef93928b"
-					(reference "C601")
+					(reference "C6001")
 					(unit 1)
 				)
@@
 		(dnp no)
 		(fields_autoplaced yes)
-		(property "Reference" "C602"
+		(property "Reference" "C6002"
 			(at 227.33 67.3565 90)
 			(effects
@@
 			(project ""
 				(path "/92ba706f-34f7-46cd-af88-2e1ff7aca489/908e7c38-dd3a-46e3-88c1-4637776bd8a8/fd7b0d96-5428-4c2c-8651-d380ef93928b"
-					(reference "C602")
+					(reference "C6002")
 					(unit 1)
 				)
@@
 		(dnp no)
 		(fields_autoplaced yes)
-		(property "Reference" "M602"
+		(property "Reference" "M6002"
 			(at 122.908 120.855 0)
 			(effects
@@
 			(project "hellenbms46"
 				(path "/92ba706f-34f7-46cd-af88-2e1ff7aca489/908e7c38-dd3a-46e3-88c1-4637776bd8a8/fd7b0d96-5428-4c2c-8651-d380ef93928b"
-					(reference "M602")
+					(reference "M6002")
 					(unit 1)
 				)
@@
 		(dnp no)
 		(fields_autoplaced yes)
-		(property "Reference" "C603"
+		(property "Reference" "C6003"
 			(at 227.33 92.7565 90)
 			(effects
@@
 			(project ""
 				(path "/92ba706f-34f7-46cd-af88-2e1ff7aca489/908e7c38-dd3a-46e3-88c1-4637776bd8a8/fd7b0d96-5428-4c2c-8651-d380ef93928b"
-					(reference "C603")
+					(reference "C6003")
 					(unit 1)
 				)
@@
 		(dnp no)
 		(fields_autoplaced yes)
-		(property "Reference" "#PWR0604"
+		(property "Reference" "#PWR06001"
 			(at 95.25 67.31 0)
 			(effects
@@
 			(project ""
 				(path "/92ba706f-34f7-46cd-af88-2e1ff7aca489/908e7c38-dd3a-46e3-88c1-4637776bd8a8/fd7b0d96-5428-4c2c-8651-d380ef93928b"
-					(reference "#PWR0604")
+					(reference "#PWR06001")
 					(unit 1)
 				)
@@
 		(dnp no)
 		(fields_autoplaced yes)
-		(property "Reference" "U601"
+		(property "Reference" "U6001"
 			(at 203.2 64.4355 0)
 			(effects
@@
 			(project ""
 				(path "/92ba706f-34f7-46cd-af88-2e1ff7aca489/908e7c38-dd3a-46e3-88c1-4637776bd8a8/fd7b0d96-5428-4c2c-8651-d380ef93928b"
-					(reference "U601")
+					(reference "U6001")
 					(unit 1)
 				)
@@
 		(dnp no)
 		(fields_autoplaced yes)
-		(property "Reference" "#PWR0606"
+		(property "Reference" "#PWR06006"
 			(at 163.83 104.14 0)
 			(effects
@@
 			(project "hellenbms46"
 				(path "/92ba706f-34f7-46cd-af88-2e1ff7aca489/908e7c38-dd3a-46e3-88c1-4637776bd8a8/fd7b0d96-5428-4c2c-8651-d380ef93928b"
-					(reference "#PWR0606")
+					(reference "#PWR06006")
 					(unit 1)
 				)
@@
 		(dnp no)
 		(fields_autoplaced yes)
-		(property "Reference" "U601"
+		(property "Reference" "U6001"
 			(at 203.2 105.8601 0)
 			(effects
@@
 			(project ""
 				(path "/92ba706f-34f7-46cd-af88-2e1ff7aca489/908e7c38-dd3a-46e3-88c1-4637776bd8a8/fd7b0d96-5428-4c2c-8651-d380ef93928b"
-					(reference "U601")
+					(reference "U6001")
 					(unit 2)
 				)
@@
 		(dnp no)
 		(fields_autoplaced yes)
-		(property "Reference" "#PWR0605"
+		(property "Reference" "#PWR06005"
 			(at 163.83 78.74 0)
 			(effects
@@
 			(project "hellenbms46"
 				(path "/92ba706f-34f7-46cd-af88-2e1ff7aca489/908e7c38-dd3a-46e3-88c1-4637776bd8a8/fd7b0d96-5428-4c2c-8651-d380ef93928b"
-					(reference "#PWR0605")
+					(reference "#PWR06005")
 					(unit 1)
 				)
@@
 		(dnp no)
 		(fields_autoplaced yes)
-		(property "Reference" "#PWR0603"
+		(property "Reference" "#PWR06002"
 			(at 95.25 148.59 0)
 			(effects
@@
 			(project ""
 				(path "/92ba706f-34f7-46cd-af88-2e1ff7aca489/908e7c38-dd3a-46e3-88c1-4637776bd8a8/fd7b0d96-5428-4c2c-8651-d380ef93928b"
-					(reference "#PWR0603")
-					(unit 1)
-				)
+					(reference "#PWR06002")
+					(unit 1)
+				)

Commit message: Initial schematic
Other:
- moved on the sheet: C6002, C6003
Changed lines of the file:
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@@
+		)
+	)
+	(bus_entry
+		(at 240.03 99.06)
+		(size 2.54 2.54)
+		(stroke
+			(width 0)
+			(type default)
+		)
+	)
+	(bus_entry
+		(at 240.03 73.66)
+		(size 2.54 2.54)
+		(stroke
+			(width 0)
+			(type default)
 		)
 	)
@@
 	(wire
 		(pts
-			(xy 213.36 99.06) (xy 223.52 99.06)
+			(xy 213.36 99.06) (xy 218.44 99.06)
 		)
 		(stroke
@@
 	(wire
 		(pts
+			(xy 226.06 73.66) (xy 240.03 73.66)
+		)
+		(stroke
+			(width 0)
+			(type default)
+		)
+	)
+	(wire
+		(pts
 			(xy 138.43 97.79) (xy 138.43 21.59)
 		)
@@
 	(wire
 		(pts
-			(xy 231.14 99.06) (xy 246.38 99.06)
-		)
-		(stroke
-			(width 0)
-			(type default)
-		)
-	)
-	(wire
-		(pts
 			(xy 58.42 45.72) (xy 72.39 45.72)
 		)
@@
 		)
 	)
-	(wire
-		(pts
-			(xy 231.14 73.66) (xy 246.38 73.66)
+	(bus
+		(pts
+			(xy 246.38 107.95) (xy 242.57 107.95)
 		)
 		(stroke
@@
 		)
 	)
+	(bus
+		(pts
+			(xy 242.57 76.2) (xy 242.57 101.6)
+		)
+		(stroke
+			(width 0)
+			(type default)
+		)
+	)
 	(wire
 		(pts
@@
 	(wire
 		(pts
+			(xy 226.06 99.06) (xy 240.03 99.06)
+		)
+		(stroke
+			(width 0)
+			(type default)
+		)
+	)
+	(wire
+		(pts
 			(xy 153.67 76.2) (xy 163.83 76.2)
 		)
@@
 		)
 	)
+	(bus
+		(pts
+			(xy 242.57 107.95) (xy 242.57 101.6)
+		)
+		(stroke
+			(width 0)
+			(type default)
+		)
+	)
 	(wire
 		(pts
@@
 	(wire
 		(pts
-			(xy 213.36 73.66) (xy 223.52 73.66)
+			(xy 213.36 73.66) (xy 218.44 73.66)
 		)
 		(stroke
@@
 			(width 0)
 			(type default)
+		)
+	)
+	(label "KNOCK_HP1"
+		(at 240.03 73.66 180)
+		(effects
+			(font
+				(size 1.27 1.27)
+			)
+			(justify right bottom)
 		)
 	)
@@
 		)
 	)
+	(label "KNOCK_HP2"
+		(at 240.03 99.06 180)
+		(effects
+			(font
+				(size 1.27 1.27)
+			)
+			(justify right bottom)
+		)
+	)
 	(label "KNOCK1"
 		(at 60.96 45.72 0)
+		(effects
+			(font
+				(size 1.27 1.27)
+			)
+			(justify left bottom)
+		)
+	)
+	(label "KNOCK_HP[1..2]"
+		(at 242.57 93.98 90)
 		(effects
 			(font
@@
 		)
 	)
-	(hierarchical_label "KNOCK_HP1"
+	(hierarchical_label "KNOCK_HP[1..2]"
 		(shape output)
-		(at 246.38 73.66 0)
+		(at 246.38 107.95 0)
 		(effects
 			(font
@@
 		(shape output)
 		(at 246.38 45.72 0)
-		(effects
-			(font
-				(size 1.27 1.27)
-			)
-			(justify left)
-		)
-	)
-	(hierarchical_label "KNOCK_HP2"
-		(shape output)
-		(at 246.38 99.06 0)
 		(effects
 			(font
@@
 	(symbol
 		(lib_id "Device:C")
-		(at 227.33 73.66 90)
+		(at 222.25 73.66 90)
 		(unit 1)
 		(exclude_from_sim no)
@@
 		(fields_autoplaced yes)
 		(property "Reference" "C6002"
-			(at 227.33 67.3565 90)
+			(at 222.25 67.3565 90)
 			(effects
 				(font
@@
 		)
 		(property "Value" "10u"
-			(at 227.33 69.7808 90)
+			(at 222.25 69.7808 90)
 			(effects
 				(font
@@
 		)
 		(property "Footprint" "Capacitor_SMD:C_0603_1608Metric"
-			(at 231.14 72.6948 0)
+			(at 226.06 72.6948 0)
 			(effects
 				(font
@@
 		)
 		(property "Datasheet" "~"
-			(at 227.33 73.66 0)
+			(at 222.25 73.66 0)
 			(effects
 				(font
@@
 		)
 		(property "Description" "Unpolarized capacitor"
-			(at 227.33 73.66 0)
+			(at 222.25 73.66 0)
 			(effects
 				(font
@@
 	(symbol
 		(lib_id "Device:C")
-		(at 227.33 99.06 90)
+		(at 222.25 99.06 90)
 		(unit 1)
 		(exclude_from_sim no)
@@
 		(fields_autoplaced yes)
 		(property "Reference" "C6003"
-			(at 227.33 92.7565 90)
+			(at 222.25 92.7565 90)
 			(effects
 				(font
@@
 		)
 		(property "Value" "10u"
-			(at 227.33 95.1808 90)
+			(at 222.25 95.1808 90)
 			(effects
 				(font
@@
 		)
 		(property "Footprint" "Capacitor_SMD:C_0603_1608Metric"
-			(at 231.14 98.0948 0)
+			(at 226.06 98.0948 0)
 			(effects
 				(font
@@
 		)
 		(property "Datasheet" "~"
-			(at 227.33 99.06 0)
+			(at 222.25 99.06 0)
 			(effects
 				(font
@@
 		)
 		(property "Description" "Unpolarized capacitor"
-			(at 227.33 99.06 0)
-			(effects
-				(font
+			(at 222.25 99.06 0)
+			(effects
+				(font

Commit message: adjusted BOM
Parts:
- C6001: footprint Capacitor_SMD:C_0603_1608Metric -> hellen-one-common:C0805; LCSC (none) -> C597285
- C6002, C6003: footprint Capacitor_SMD:C_0603_1608Metric -> hellen-one-common:C0805; LCSC (none) -> C440198
- U6001: LCSC (none) -> C636235
Changed lines of the file:
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@@
+			)
+		)
+		(property "LCSC" "C636235"
+			(at 166.37 86.36 0)
+			(effects
+				(font
+					(size 1.27 1.27)
+				)
+				(hide yes)
 			)
 		)
@@
 			)
 		)
-		(property "Footprint" "Capacitor_SMD:C_0603_1608Metric"
+		(property "Footprint" "hellen-one-common:C0805"
 			(at 154.6352 90.17 0)
 			(effects
@@
 			)
 		)
+		(property "LCSC" "C597285"
+			(at 153.67 86.36 0)
+			(effects
+				(font
+					(size 1.27 1.27)
+				)
+				(hide yes)
+			)
+		)
 		(pin "1"
 		)
@@
 			)
 		)
-		(property "Footprint" "Capacitor_SMD:C_0603_1608Metric"
+		(property "Footprint" "hellen-one-common:C0805"
 			(at 226.06 72.6948 0)
 			(effects
@@
 			)
 		)
+		(property "LCSC" "C440198"
+			(at 222.25 73.66 0)
+			(effects
+				(font
+					(size 1.27 1.27)
+				)
+				(hide yes)
+			)
+		)
 		(pin "1"
 		)
@@
 		(fields_autoplaced yes)
 		(property "Reference" "C6003"
-			(at 222.25 92.7565 90)
+			(at 222.25 91.44 90)
 			(effects
 				(font
@@
 		)
 		(property "Value" "10u"
-			(at 222.25 95.1808 90)
-			(effects
-				(font
-					(size 1.27 1.27)
-				)
-			)
-		)
-		(property "Footprint" "Capacitor_SMD:C_0603_1608Metric"
+			(at 222.25 93.98 90)
+			(effects
+				(font
+					(size 1.27 1.27)
+				)
+			)
+		)
+		(property "Footprint" "hellen-one-common:C0805"
 			(at 226.06 98.0948 0)
 			(effects
@@
 			)
 		)
+		(property "LCSC" "C440198"
+			(at 222.25 99.06 0)
+			(effects
+				(font
+					(size 1.27 1.27)
+				)
+				(hide yes)
+			)
+		)
 		(pin "1"
 		)
@@
 		)
 		(property "Description" "1MHz, Low-Power Op Amp, SOIC-8"
+			(at 203.2 73.66 0)
+			(effects
+				(font
+					(size 1.27 1.27)
+				)
+				(hide yes)
+			)
+		)
+		(property "LCSC" "C636235"
 			(at 203.2 73.66 0)
 			(effects
@@
 			(at 203.2 99.06 0)
 			(effects
+				(font
+					(size 1.27 1.27)
+				)
+				(hide yes)
+			)
+		)
+		(property "LCSC" "C636235"
+			(at 203.2 99.06 0)
+			(effects
