File: nbo2h.kicad_sch (KiCad schematic)
At the start: 3 parts, among them Q11001 ISL9V3040D3ST

Commit message: adjusted BOM
Parts:
- Q11001: LCSC (none) -> C462128
Changed lines of the file:
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@@
 			)
 		)
-		(property "LCSC" ""
+		(property "LCSC" "C462128"
 			(at 147.32 72.39 0)
 			(effects
