File: hellenbms46.kicad_pcb (KiCad board)
At the start: 4 copper layers, 164 x 118 mm, 40 parts, among them J201 Conn_02x03_Top_Bottom, J203 Conn_02x12_Top_Bottom, J301 USB_B, M301 Module:mega-mcu100/0.3, M302 Module-can-0.1, M303 Module-wbo-0.5, M304 Module-lin-0.1, M306 Module-power_12and5V-0.2, M601 Module-knock-0.2, M602 Module-knock-0.2, P201 134pin_7-967288-1_KC5, Q401 ISL9V3040D3ST, Q402 ISL9V3040D3ST, Q403 ISL9V3040D3ST, Q404 ISL9V3040D3ST, U501 VNLD5160TR-E, U502 VNLD5160TR-E, U601 MCP6002-xSN

Commit message: test commit
Parts:
- renumbered BT301 to BT3001, C601 to C6001, C602 to C6002, C603 to C6003, D301 to D3001, F401 to F4001, F403 to F4002, F404 to F4003, F402 to F4004, J203 to J2001, J201 to J2002, J301 to J3001, JP301 to JP3001, M306 to M3001, M301 to M3002, M302 to M3003, M303 to M3004, M304 to M3005, M601 to M6001, M602 to M6002, P201 to P2001, Q401 to Q4001, Q403 to Q4002, Q404 to Q4003, Q402 to Q4004, R403 to R4001, R406 to R4002, R408 to R4003, R401 to R4004, R405 to R4005, R407 to R4006, R404 to R4007, R402 to R4008, R502 to R5001, R504 to R5002, R501 to R5003, R503 to R5004, U501 to U5001, U502 to U5002, U601 to U6001

Commit message: Initial schematic
Parts:
- removed the R4004 at (97.5, 73.6)
- removed R4005, R4006, R4008: 0, Resistor_SMD:R_2512_6332Metric
- added C10001: 10u, hellen-one-common:C0805, F.Cu at (140.8, 86.4)
- added C10002: 10n, hellen-one-common:C0805, F.Cu at (143.1, 86.4)
- added C10003: 10n, hellen-one-common:C0805, F.Cu at (145.3, 86.4)
- added C9001: 10u, hellen-one-common:C0805, F.Cu at (199.1, 103.8)
- added C9002: 10n, hellen-one-common:C0805, F.Cu at (199.1, 108.3)
- added C9003: 10n, hellen-one-common:C0805, F.Cu at (199.1, 106.0)
- added F11001: 50mA, Fuse:Fuse_0603_1608Metric, F.Cu at (106.0, 127.5)
- added F2001: 10A, hellen-one-common:36911600000, F.Cu at (126.0, 75.0)
- added F2002: 10A, hellen-one-common:36911600000, F.Cu at (112.5, 75.0)
- added F2003: 10A, hellen-one-common:36911600000, F.Cu at (121.5, 75.0)
- added F2004: 10A, hellen-one-common:36911600000, F.Cu at (117.0, 75.0)
- added JP2001: Jumper_2_Bridged, Jumper:SolderJumper-2_P1.3mm_Bridged_RoundedPad1.0x1.5mm, F.Cu at (188.0, 71.7)
- added JP2002: Jumper_2_Open, hellen-one-common:PAD-0805-PAD, F.Cu at (193.0, 71.0)
- added JP2003: Jumper_2_Bridged, Jumper:SolderJumper-2_P1.3mm_Bridged_RoundedPad1.0x1.5mm, F.Cu at (200.5, 74.5)
- added JP2004: Jumper_2_Bridged, Jumper:SolderJumper-2_P1.3mm_Bridged_RoundedPad1.0x1.5mm, F.Cu at (200.5, 71.0)
- added JP2005: Jumper_2_Bridged, Jumper:SolderJumper-2_P1.3mm_Bridged_RoundedPad1.0x1.5mm, F.Cu at (146.5, 73.0)
- added JP2006: Jumper_2_Open, hellen-one-common:PAD-0805-PAD, F.Cu at (162.6, 73.0)
- added JP2007: Jumper_2_Open, hellen-one-common:PAD-0805-PAD, F.Cu at (159.7, 73.0)
- added JP2008: Jumper_2_Open, hellen-one-common:PAD-0805-PAD, F.Cu at (156.9, 73.0)
- added JP2009: Jumper_2_Open, hellen-one-common:PAD-0805-PAD, F.Cu at (154.0, 73.0)
- added JP2010: Jumper_2_Bridged, Jumper:SolderJumper-2_P1.3mm_Bridged_RoundedPad1.0x1.5mm, F.Cu at (144.0, 73.0)
- added JP2011: Jumper_2_Bridged, Jumper:SolderJumper-2_P1.3mm_Bridged_RoundedPad1.0x1.5mm, F.Cu at (133.5, 73.2)
- added JP2012: Jumper_2_Bridged, Jumper:SolderJumper-2_P1.3mm_Bridged_RoundedPad1.0x1.5mm, F.Cu at (131.0, 73.2)
- added JP4001: Jumper_2_Open, hellen-one-common:PAD-0805-PAD, F.Cu at (98.5, 75.5)
- added JP4002: Jumper_2_Open, hellen-one-common:PAD-0805-PAD, F.Cu at (98.5, 88.0)
- added JP4003: Jumper_2_Open, hellen-one-common:PAD-0805-PAD, F.Cu at (98.5, 99.2)
- added JP4004: Jumper_2_Open, hellen-one-common:PAD-0805-PAD, F.Cu at (99.0, 110.5)
- added Q11001: ISL9V3040D3ST, Package_TO_SOT_SMD:TO-252-2, F.Cu at (94.5, 127.7)
- added R10001: 1k, hellen-one-common:R0603, F.Cu at (140.7, 90.1)
- added R10002: 1k, hellen-one-common:R0603, F.Cu at (142.7, 90.1)
- added R10003: 10k, hellen-one-common:R0603, F.Cu at (144.6, 90.1)
- added R10004: 10k, hellen-one-common:R0603, F.Cu at (146.5, 90.1)
- added R11001: 22, hellen-one-common:R0603, F.Cu at (103.0, 128.2)
- added R7001: 4.7k, hellen-one-common:R0603, F.Cu at (203.4, 85.6)
- added R7002: 4.7k, hellen-one-common:R0603, F.Cu at (182.8, 94.3)
- added R7003: 4.7k, hellen-one-common:R0603, F.Cu at (203.8, 89.5)
- added R7004: 4.7k, hellen-one-common:R0603, F.Cu at (183.3, 96.8)
- added R8001: 4.7k, hellen-one-common:R0603, F.Cu at (150.3, 169.5)
- added R8002: 4.7k, hellen-one-common:R0603, F.Cu at (122.8, 166.0)
- added R8003: 4.7k, hellen-one-common:R0603, F.Cu at (150.3, 173.0)
- added R8004: 4.7k, hellen-one-common:R0603, F.Cu at (123.0, 163.5)
- added R9001: 1k, hellen-one-common:R0603, F.Cu at (195.4, 103.6)
- added R9002: 1k, hellen-one-common:R0603, F.Cu at (195.4, 105.6)
- added R9003: 10k, hellen-one-common:R0603, F.Cu at (195.4, 107.5)
- added R9004: 10k, hellen-one-common:R0603, F.Cu at (195.4, 109.5)
- added REF**: MountingHole_4mm_Pad, MountingHole:MountingHole_4mm_Pad, F.Cu at (83.5, 44.0)
- added REF**: MountingHole_4mm_Pad, MountingHole:MountingHole_4mm_Pad, F.Cu at (88.0, 154.0)
- added REF**: MountingHole_4mm_Pad, MountingHole:MountingHole_4mm_Pad, F.Cu at (236.0, 154.0)
- added REF**: MountingHole_4mm_Pad, MountingHole:MountingHole_4mm_Pad, F.Cu at (240.5, 44.0)
- added TP3001: TestPoint, TestPoint:TestPoint_Keystone_5000-5004_Miniature, F.Cu at (66.7, 146.7)
- added TP3002: TestPoint, TestPoint:TestPoint_Keystone_5000-5004_Miniature, F.Cu at (66.7, 129.3)
- added TP3003: TestPoint, TestPoint:TestPoint_Keystone_5000-5004_Miniature, F.Cu at (66.7, 133.7)
- added TP3004: TestPoint, TestPoint:TestPoint_Keystone_5000-5004_Miniature, F.Cu at (66.7, 138.0)
- added TP3005: TestPoint, TestPoint:TestPoint_Keystone_5000-5004_Miniature, F.Cu at (66.7, 142.3)
- added TP3006: TestPoint, TestPoint:TestPoint_Keystone_5000-5004_Miniature, F.Cu at (71.0, 133.7)
- added TP3007: TestPoint, TestPoint:TestPoint_Keystone_5000-5004_Miniature, F.Cu at (71.0, 129.3)
- added TP3008: TestPoint, TestPoint:TestPoint_Keystone_5000-5004_Miniature, F.Cu at (71.0, 146.7)
- added TP3009: TestPoint, TestPoint:TestPoint_Keystone_5000-5004_Miniature, F.Cu at (71.0, 138.0)
- added TP3010: TestPoint, TestPoint:TestPoint_Keystone_5000-5004_Miniature, F.Cu at (71.0, 142.3)
- added U10001: TC4427xOA, Package_SO:SOIC-8_3.9x4.9mm_P1.27mm, F.Cu at (136.0, 87.5)
- added U7001: VNLD5160TR-E, Package_SO:SOIC-8_3.9x4.9mm_P1.27mm, F.Cu at (197.5, 88.0)
- added U7002: VNLD5160TR-E, Package_SO:SOIC-8_3.9x4.9mm_P1.27mm, F.Cu at (177.0, 96.4)
- added U8001: VNLD5160TR-E, Package_SO:SOIC-8_3.9x4.9mm_P1.27mm, F.Cu at (144.5, 171.9)
- added U8002: VNLD5160TR-E, Package_SO:SOIC-8_3.9x4.9mm_P1.27mm, F.Cu at (117.5, 165.5)
- added U9001: TC4427xOA, Package_SO:SOIC-8_3.9x4.9mm_P1.27mm, F.Cu at (198.0, 99.4)
- moved M3005 81.2 mm to (117.2, 103.2)
- moved M3003 46.7 mm to (154.2, 135.1), turned to 180 degrees
- moved J2001 36.1 mm to (176.5, 138.7)
- moved M3004 29.5 mm to (186.9, 130.2), turned to 90 degrees
- moved M3002 24.9 mm to (168.4, 129.9), turned to 90 degrees
- moved C6001 12.0 mm to (187.2, 80.6)
- moved C6002 12.0 mm to (179.8, 79.0)
- moved U6001 12.0 mm to (181.5, 82.5)
- moved C6003 12.0 mm to (187.2, 83.1)
- moved F4004 9.98 mm to (106.4, 115.5)
- moved Q4004 9.98 mm to (94.7, 115.5)
- moved R4004 9.98 mm to (103.8, 116.3)
- moved M6002 6.85 mm to (172.3, 72.0), turned to -90 degrees
- moved J3001 6.79 mm to (216.5, 149.6)
- moved F4003 6.26 mm to (106.4, 104.2)
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- renumbered M3004 to M3003, M3003 to M3004, R4007 to R4004
Connections:
- net /rusefi/Ignition/IN1 renamed /rusefi/IGN1
- net /rusefi/Ignition/IN2 renamed /rusefi/IGN2
- net /rusefi/Ignition/IN3 renamed /rusefi/IGN3
- net /rusefi/Ignition/IN4 renamed /rusefi/IGN4
- net /rusefi/Injection/IN1 renamed /rusefi/INJ1
- net /rusefi/Injection/IN2 renamed /rusefi/INJ2
- net /rusefi/Injection/IN3 renamed /rusefi/INJ3
- net /rusefi/Injection/IN4 renamed /rusefi/INJ4
- J2001 pad 1: unconnected-(J2001-Pin_1-Pad1) -> /rusefi/USB.DP
- J2001 pad 11: unconnected-(J2001-Pin_11-Pad11) -> /rusefi/USB.VBUS
- J2001 pad 12: unconnected-(J2001-Pin_12-Pad12) -> GND
- J2001 pad 13: unconnected-(J2001-Pin_13-Pad13) -> /rusefi/CAN2L
- J2001 pad 14: unconnected-(J2001-Pin_14-Pad14) -> /rusefi/CAN2H
- J2001 pad 15: unconnected-(J2001-Pin_15-Pad15) -> /rusefi/KnockAmps/KNOCK_HP2
- J2001 pad 16: unconnected-(J2001-Pin_16-Pad16) -> GND
- J2001 pad 17: unconnected-(J2001-Pin_17-Pad17) -> GND
- J2001 pad 18: unconnected-(J2001-Pin_18-Pad18) -> /rusefi/AIN.MAP
- J2001 pad 19: unconnected-(J2001-Pin_19-Pad19) -> +5VA
- J2001 pad 2: unconnected-(J2001-Pin_2-Pad2) -> /rusefi/USB.DM
- J2001 pad 20: unconnected-(J2001-Pin_20-Pad20) -> +5VA
- J2001 pad 21: unconnected-(J2001-Pin_21-Pad21) -> GND
- J2001 pad 3: unconnected-(J2001-Pin_3-Pad3) -> /rusefi/CAN1L
- J2001 pad 4: unconnected-(J2001-Pin_4-Pad4) -> /rusefi/CAN1H
- J2001 pad 5: unconnected-(J2001-Pin_5-Pad5) -> /rusefi/KnockAmps/KNOCK_HP1
- J2001 pad 6: unconnected-(J2001-Pin_6-Pad6) -> +12V_RAW
- J2001 pad 7: unconnected-(J2001-Pin_7-Pad7) -> GND
- M3002 pad E10: unconnected-(M3002-OUT_INJ8_(PD12)-PadE10) -> /rusefi/OUT LS1/IN4
- M3002 pad E11: unconnected-(M3002-OUT_INJ7_(PD15)-PadE11) -> /rusefi/OUT LS1/IN3
- M3002 pad E12: unconnected-(M3002-OUT_INJ6_(PA8)-PadE12) -> /rusefi/OUT LS1/IN2
- M3002 pad E13: unconnected-(M3002-OUT_INJ5_(PD2)-PadE13) -> /rusefi/OUT LS1/IN1
- M3002 pad E18: unconnected-(M3002-OUT_PWM1_(PD13)-PadE18) -> /rusefi/OUT PP/IN1
- M3002 pad E19: unconnected-(M3002-OUT_PWM2_(PC6)-PadE19) -> /rusefi/OUT PP/IN2
- M3002 pad E20: unconnected-(M3002-OUT_PWM3_(PC7)-PadE20) -> /rusefi/OUT PP1/IN1
- M3002 pad E21: unconnected-(M3002-OUT_PWM4_(PC8)-PadE21) -> /rusefi/OUT PP1/IN2
- M3002 pad E22: unconnected-(M3002-OUT_PWM5_(PC9)-PadE22) -> /rusefi/NBO2H/IN
- M3002 pad E23: unconnected-(M3002-OUT_PWM6_(PD14)-PadE23) -> Net-(M3002-OUT_PWM6_(PD14))
- M3002 pad N16: unconnected-(M3002-BOOT0-PadN16) -> Net-(M3002-BOOT0)
- M3002 pad N4: unconnected-(M3002-USBID_(PA10)-PadN4) -> Net-(M3002-USBID_(PA10))
- M3002 pad N7: unconnected-(M3002-nReset-PadN7) -> Net-(M3002-nReset)
- M3002 pad S1: unconnected-(M3002-IN_D4_(PE15)-PadS1) -> /rusefi/EXTIN2
- M3002 pad S10: unconnected-(M3002-IN_O2S2_(PA1)-PadS10) -> /rusefi/AIN.NBO2
- M3002 pad S11: unconnected-(M3002-IN_O2S_/_CAN_WAKEUP_(PA0)-PadS11) -> Net-(M3002-IN_O2S_/_CAN_WAKEUP_(PA0))
- M3002 pad S12: unconnected-(M3002-IN_MAP2_(PC1)-PadS12) -> Net-(M3002-IN_MAP2_(PC1))
- M3002 pad S14: unconnected-(M3002-IN_CRANK_(PB1)-PadS14) -> /rusefi/DIN.CPS
- M3002 pad S16: unconnected-(M3002-IN_CAM_(PA6)-PadS16) -> /rusefi/DIN.CMP
- M3002 pad S17: unconnected-(M3002-IN_VSS_(PE11)-PadS17) -> /rusefi/DIN.RRWS
- M3002 pad S19: unconnected-(M3002-IN_PPS_(PA3)-PadS19) -> Net-(M3002-IN_PPS_(PA3))
- M3002 pad S2: unconnected-(M3002-IN_D3_(PE14)-PadS2) -> /rusefi/EXTIN1
- M3002 pad S3: unconnected-(M3002-IN_D2_(PE13)-PadS3) -> /rusefi/DIN.EWS
- M3002 pad S4: unconnected-(M3002-IN_D1_(PE12)-PadS4) -> /rusefi/DIN.OPS
- M3002 pad S5: unconnected-(M3002-VREF2-PadS5) -> Net-(M3002-VREF2)
- M3002 pad S6: unconnected-(M3002-IN_AUX4_(PC5)-PadS6) -> Net-(M3002-IN_AUX4_(PC5))
- M3002 pad S8: /rusefi/AIN.OILTEMP2 -> /rusefi/AIN.TRAD
- M3002 pad S9: /rusefi/AIN.OILTEMP1 -> /rusefi/AIN.MAF
- M3002 pad W11: /rusefi/CANH -> /rusefi/CAN1H
- M3002 pad W12: /rusefi/CANL -> /rusefi/CAN1L
- M3002 pad W13: unconnected-(M3002-V33_REF-PadW13) -> Net-(M3002-V33_REF)
- M3002 pad W3: unconnected-(M3002-IGN8_(PE6)-PadW3) -> /rusefi/OUT LS/IN4
- M3002 pad W4: unconnected-(M3002-IGN7_(PB9)-PadW4) -> /rusefi/OUT LS/IN3
- M3002 pad W5: unconnected-(M3002-IGN6_(PB8)-PadW5) -> /rusefi/OUT LS/IN2
- M3002 pad W6: unconnected-(M3002-IGN5_(PE2)-PadW6) -> /rusefi/OUT LS/IN1
- M3003 pad W1: unconnected-(M3004-V5_IN-PadW1) -> +5VA
- M3003 pad W3: /rusefi/CANL -> /rusefi/CAN1L
- M3003 pad W4: /rusefi/CANH -> /rusefi/CAN1H
- M3004 pad S1: unconnected-(M3003-CANL-PadS1) -> /rusefi/CAN2L
- M3004 pad S2: unconnected-(M3003-CANH-PadS2) -> /rusefi/CAN2H
- M3004 pad V1: unconnected-(M3003-V5-PadV1) -> +5VA
- M3005 pad V3: unconnected-(M3005-5V-PadV3) -> +5VA
- M3005 pad V4: /conn/LIN -> /rusefi/LIN
- P2001 pad 206: /conn/LIN -> /conn/ECU_LIN
- P2001 pad 224: /conn/ECU_NBO2pre_H+ -> +12V_RAW
- P2001 pad 303: unconnected-(P2001C-Pin_303-Pad303) -> +12V_RAW
- P2001 pad 304: unconnected-(P2001C-Pin_304-Pad304) -> +12V_RAW
- P2001 pad 305: unconnected-(P2001C-Pin_305-Pad305) -> +12V_RAW
- P2001 pad 306: unconnected-(P2001C-Pin_306-Pad306) -> +12V_RAW
- P2001 pad 307: GND -> /conn/OUTLS.SLV
- P2001 pad 309: GND -> /conn/OUTLS.THERMO
- P2001 pad 312: unconnected-(P2001C-Pin_312-Pad312) -> /conn/CRANK_FB
- P2001 pad 313: unconnected-(P2001C-Pin_313-Pad313) -> /conn/CHARGE
- P2001 pad 316: unconnected-(P2001C-Pin_316-Pad316) -> +12V_RAW
- P2001 pad 326: unconnected-(P2001C-Pin_326-Pad326) -> /conn/OIL_P
- P2001 pad 327: unconnected-(P2001C-Pin_327-Pad327) -> +5VA
- P2001 pad 328: unconnected-(P2001C-Pin_328-Pad328) -> /rusefi/AIN.CLT
- P2001 pad 329: unconnected-(P2001C-Pin_329-Pad329) -> /rusefi/AIN.IAT
- P2001 pad 330: unconnected-(P2001C-Pin_330-Pad330) -> /rusefi/AIN.MAF
- P2001 pad 331: /conn/KNOCK1 -> /conn/KNOCK2
- P2001 pad 332: /conn/KNOCK2 -> /conn/KNOCK1
- P2001 pad 333: unconnected-(P2001C-Pin_333-Pad333) -> /rusefi/AIN.TPS
- P2001 pad 335: unconnected-(P2001C-Pin_335-Pad335) -> /rusefi/DIN.CPS
- P2001 pad 338: unconnected-(P2001C-Pin_338-Pad338) -> /rusefi/DIN.CMP
- P2001 pad 339: unconnected-(P2001C-Pin_339-Pad339) -> /conn/F_OLN
- P2001 pad 340: unconnected-(P2001C-Pin_340-Pad340) -> /conn/PP.IACVO
- P2001 pad 341: unconnected-(P2001C-Pin_341-Pad341) -> /conn/PP.IACVC
- P2001 pad 343: unconnected-(P2001C-Pin_343-Pad343) -> +12V_RAW
- P2001 pad 344: unconnected-(P2001C-Pin_344-Pad344) -> /conn/OUTLS.FTVV
- P2001 pad 345: unconnected-(P2001C-Pin_345-Pad345) -> /conn/OUTLS.DISA
- P2001 pad 346: unconnected-(P2001C-Pin_346-Pad346) -> +5VA
- P2001 pad 348: /conn/INJ_OUT4 -> Net-(P2001C-Pin_348)
- P2001 pad 349: /conn/INJ_OUT3 -> Net-(P2001C-Pin_349)
- P2001 pad 350: /conn/INJ_OUT2 -> Net-(P2001C-Pin_350)
- P2001 pad 351: /conn/INJ_OUT1 -> Net-(P2001C-Pin_351)
- P2001 pad 352: unconnected-(P2001C-Pin_352-Pad352) -> +12V_RAW
- P2001 pad 401: unconnected-(P2001D-Pin_401-Pad401) -> /conn/CHARGE
- P2001 pad 402: unconnected-(P2001D-Pin_402-Pad402) -> /conn/CRANK_FB
- P2001 pad 403: unconnected-(P2001D-Pin_403-Pad403) -> /conn/OUTLS.SLP
- P2001 pad 404: unconnected-(P2001D-Pin_404-Pad404) -> /conn/PP.FAN
- P2001 pad 410: unconnected-(P2001D-Pin_410-Pad410) -> /conn/OUTLS.EKP
- P2001 pad 411: unconnected-(P2001D-Pin_411-Pad411) -> /conn/OIL_P
- P2001 pad 417: unconnected-(P2001D-Pin_417-Pad417) -> /conn/PP.FTD
- P2001 pad 421: unconnected-(P2001D-Pin_421-Pad421) -> /conn/F_OLN
- P2001 pad 422: unconnected-(P2001D-Pin_422-Pad422) -> /rusefi/DIN.RRWS
- P2001 pad 429: unconnected-(P2001D-Pin_429-Pad429) -> /conn/OUTLS.KOREL
- P2001 pad 432: /conn/LIN -> /conn/ECU_LIN
- P2001 pad 433: unconnected-(P2001D-Pin_433-Pad433) -> /rusefi/DIN.EWS
- P2001 pad 439: unconnected-(P2001D-Pin_439-Pad439) -> /rusefi/AIN.TRAD
- P2001 pad 504: /conn/IGN_OUT2 -> Net-(P2001E-Pin_504)
- P2001 pad 506: /conn/IGN_OUT1 -> Net-(P2001E-Pin_506)
- P2001 pad 508: /conn/IGN_OUT3 -> Net-(P2001E-Pin_508)
- P2001 pad 509: /conn/IGN_OUT4 -> Net-(P2001E-Pin_509)

Commit message: inital schamatic
Connections:
- J2001 pad 22: unconnected-(J2001-Pin_22-Pad22) -> /conn/EXTIN1
- J2001 pad 23: unconnected-(J2001-Pin_23-Pad23) -> /conn/EXTIN2
- J2002 pad 1: unconnected-(J2002-Pin_1-Pad1) -> +12V_RAW
- M3001 pad S1: unconnected-(M3001-GND-PadS1) -> GND
- M3002 pad S1: /rusefi/EXTIN2 -> /conn/EXTIN2
- M3002 pad S2: /rusefi/EXTIN1 -> /conn/EXTIN1
- M3003 pad E6: unconnected-(M3003-LSU_H--PadE6) -> GND
- M3003 pad G: unconnected-(M3003-GND-PadG) -> GND
- M3004 pad E1: unconnected-(M3004-GND-PadE1) -> GND
- M3004 pad V2: unconnected-(M3004-CAN_VIO-PadV2) -> +3.3VA
- M3005 pad E1: unconnected-(M3005-GND-PadE1) -> GND
- M3005 pad N1: unconnected-(M3005-12V-PadN1) -> +12V_RAW
- M3005 pad S1: unconnected-(M3005-GND-PadS1) -> GND
- M3005 pad V1: unconnected-(M3005-12V-PadV1) -> +12V_RAW

Commit message: testsing
Parts:
- C6001, C6002, C6003: footprint Capacitor_SMD:C_0603_1608Metric -> hellen-one-common:C0805
- moved TP3005 118.1 mm to (178.0, 103.0)
- moved TP3004 111.7 mm to (174.0, 107.0)
- moved TP3003 108.8 mm to (174.5, 119.0)
- moved TP3002 107.9 mm to (173.5, 114.5)
- moved TP3006 102.9 mm to (173.5, 124.5)
- moved TP3008 77.3 mm to (128.5, 95.0)
- moved TP3007 76.0 mm to (138.0, 93.5)
- moved TP3001 73.6 mm to (139.0, 133.0)
- moved R8001 72.1 mm to (205.9, 123.5)
- moved R8003 72.1 mm to (205.9, 127.0)
- moved U8001 72.1 mm to (200.0, 125.9)
- moved TP3009 67.4 mm to (127.0, 100.5)
- moved TP3010 61.2 mm to (125.5, 114.5)
- moved U8002 39.1 mm to (119.5, 126.4)
- moved R8002 39.1 mm to (124.8, 126.9)
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